File: hank-hill-sao.kicad_pcb (KiCad board)
At the start: 2 copper layers, 60.2 x 98.3 mm, 3 parts

Commit message: updated
Parts:
- removed the G*** at (0.00, 0.00) (x3)
- added D1: LED, LED_SMD:LED_1206_3216Metric, B.Cu at (-14.5, -3.73)
- added D2: LED, LED_SMD:LED_1206_3216Metric, B.Cu at (11.3, -4.10)
- added G*** (x5): LOGO, LOGO, F.Cu at (0.00, 0.00)
- added R1: 1K, Resistor_SMD:R_1206_3216Metric, B.Cu at (-1.52, 6.37)
- added X1: Badgelife_sao_connector_v169bis, my-ki-cad-parts:Badgelife-SAOv169-SAO-2x3, F.Cu at (-1.09, 36.2)
Routing:
- net Net-(D1-Pad2): track 0.00 -> 38.2 mm
- net /VDD: track 0.00 -> 30.0 mm
- added copper zone on B.Cu, net GND

Commit message: final and ready for fab
Parts:
- removed the G*** at (0.00, 0.00) (x5)
- added G*** (x6): LOGO, LOGO, F.Cu at (0.00, 0.00)
- moved D2 25.9 mm to (-14.6, -3.95), turned to 180 degrees
- moved D1 25.4 mm to (10.9, -3.75), turned to 180 degrees
- moved R1 5.44 mm to (-2.00, 11.8), turned to 180 degrees
- moved X1 4.83 mm to (-1.08, 41.1)
Routing:
- net Net-(D1-Pad2): track 38.2 -> 44.1 mm
- net /VDD: track 30.0 -> 28.1 mm
